Commit message: refactor urdf; add mover_pcb

File: ros_ws/src/mover_description/urdf/mover.urdf.xacro (robot description, xacro)
@@ -2,4 +2,5 @@
 <robot xmlns:xacro="http://www.ros.org/wiki/xacro" name="mover">
         <link name="world"></link>
+        <xacro:include filename="wheel.xacro"/>
         <!-- Main Chassis -->
         <joint name="base_joint" type="fixed">
@@ -29,89 +30,3 @@
                 </inertial>
         </link>
-        <!-- The front roller -->
-        <joint name="roller_joint" type="fixed">
-                <parent link="base_link"/>
-                <child link="roller_link"/>
-                <origin xyz="0 -0.12 -0.04" rpy="0 0 0"/>
-        </joint>
-        <link name="roller_link">
-                <visual>
-                        <origin xyz="0 0 0" rpy="0 0 0"/>
-                        <geometry>
-                                <sphere radius="0.02"/>
-                        </geometry>
-                        <material name="black">
-                                <color rgba="0 0 0 1"/>
-                        </material>
-                </visual>
-                <collision>
-                        <origin xyz="0 0 0" rpy="0 0 0"/>
-                        <geometry>
-                                <sphere radius="0.02"/>
-                        </geometry>
-                </collision>
-                <inertial>
-                        <origin xyz="0 0 0" rpy="0 0 0"/>
-                        <mass value="0.1"/>
-                                <inertia ixx="0.0082" ixy="0.0" ixz="0.0" iyy="0.0082" iyz="0.0" izz="0.0154" />
-                </inertial>
-        </link>
-        <!-- Right wheel -->
-        <joint name="wheel_right_joint" type="continuous">
-                <parent link="base_link"/>
-                <child link="wheel_right_link"/>
-                <origin xyz="-0.11 0 -0.03" rpy="0 1.57075 0"/>
-                <axis xyz="0 0 1"/>
-        </joint>
-        <link name="wheel_right_link">
-                <visual>
-                        <origin xyz="0 0 0" rpy="0 0 0"/>
-                        <geometry>
-                                <cylinder length="0.016" radius="0.033"/>
-                        </geometry>
-                        <material name="black">
-                                <color rgba="0 0 0 1"/>
-                        </material>
-                </visual>
-                <collision>
-                        <origin xyz="0 0 0" rpy="0 0 0"/>
-                        <geometry>
-                                <cylinder length="0.016" radius="0.033"/>
-                        </geometry>
-                </collision>
-                <inertial>
-                        <origin xyz="0 0 0" rpy="0 0 0"/>
-                        <mass value="0.2"/>
-                                <inertia ixx="0.0082" ixy="0.0" ixz="0.0" iyy="0.0082" iyz="0.0" izz="0.0154" />
-                </inertial>
-        </link>
-        <!-- Left wheel -->
-        <joint name="wheel_left_joint" type="continuous">
-                <parent link="base_link"/>
-                <child link="wheel_left_link"/>
-                <origin xyz="0.11 0 -0.03" rpy="0 1.57075 0"/>
-                <axis xyz="0 0 1"/>
-        </joint>
-        <link name="wheel_left_link">
-                <visual>
-                        <origin xyz="0 0 0" rpy="0 0 0"/>
-                        <geometry>
-                                <cylinder length="0.016" radius="0.033"/>
-                        </geometry>
-                        <material name="black">
-                                <color rgba="0 0 0 1"/>
-                        </material>
-                </visual>
-                <collision>
-                        <origin xyz="0 0 0" rpy="0 0 0"/>
-                        <geometry>
-                                <cylinder length="0.016" radius="0.033"/>
-                        </geometry>
-                </collision>
-                <inertial>
-                        <origin xyz="0 0 0" rpy="0 0 0"/>
-                        <mass value="0.2"/>
-                                <inertia ixx="0.0082" ixy="0.0" ixz="0.0" iyy="0.0082" iyz="0.0" izz="0.0154" />
-                </inertial>
-        </link>
 </robot>

Commit message: fix controller

File: ros_ws/src/mover_description/urdf/mover.urdf.xacro (robot description, xacro)
@@ -2,7 +2,6 @@
 <robot xmlns:xacro="http://www.ros.org/wiki/xacro" name="mover">
         <link name="world"></link>
-        <xacro:include filename="wheel.xacro"/>
-        <!-- Main Chassis -->
         <joint name="base_joint" type="fixed">
+                <origin xyz="0 0 0" rpy="0 0 0"/>
                 <parent link="world"/>
                 <child link="base_link"/>
@@ -14,6 +13,6 @@
                                 <cylinder length="0.07" radius="0.16"/>
                         </geometry>
-                        <material name="green">
-                                <color rgba="0 1 0 1"/>
+                        <material>
+                                <color rgba="0.5 0.5 0.5 1"/>
                         </material>
                 </visual>
@@ -27,5 +26,5 @@
                         <origin xyz="0 0 0" rpy="0 0 0"/>
                         <mass value="1.2"/>
-                                <inertia ixx="0.0082" ixy="0.0" ixz="0.0" iyy="0.0082" iyz="0.0" izz="0.0154" />
+                        <inertia ixx="2.26" ixy="0.0" ixz="0.0" iyy="6.26" iyz="0.0" izz="8.5" />
                 </inertial>
         </link>

Commit message: add urdf launch for rviz

File: ros_ws/src/mover_description/urdf/mover.urdf.xacro (robot description, xacro)
@@ -1,4 +1,5 @@
 <?xml version="1.0"?>
 <robot xmlns:xacro="http://www.ros.org/wiki/xacro" name="mover">
+        <xacro:include filename="wheel.xacro" />
         <link name="world"></link>
         <joint name="base_joint" type="fixed">
@@ -13,5 +14,5 @@
                                 <cylinder length="0.07" radius="0.16"/>
                         </geometry>
-                        <material>
+                        <material name="gray">
                                 <color rgba="0.5 0.5 0.5 1"/>
                         </material>

File: ros_ws/src/mover_description/urdf/wheel.xacro (robot description, xacro)
@@ -1,40 +1,41 @@
 <?xml version="1.0"?>
 <robot xmlns:xacro="http://www.ros.org/wiki/xacro">
-        <!-- The front roller -->
-        <joint name="roller_joint" type="fixed">
+<!-- The front roller -->
+<joint name="roller_joint" type="fixed">
+        <parent link="base_link"/>
+        <child link="roller_link"/>
+        <origin xyz="0 -0.12 -0.04" rpy="0 0 0"/>
+</joint>
+<link name="roller_link">
+        <visual>
+                <origin xyz="0 0 0" rpy="0 0 0"/>
+                <geometry>
+                        <sphere radius="0.02"/>
+                </geometry>
+                <material name="black">
+                        <color rgba="0 0 0 1"/>
+                </material>
+        </visual>
+        <collision>
+                <origin xyz="0 0 0" rpy="0 0 0"/>
+                <geometry>
+                        <sphere radius="0.02"/>
+                </geometry>
+        </collision>
+        <inertial>
+                <origin xyz="0 0 0" rpy="0 0 0"/>
+                <mass value="0.1"/>
+                <inertia ixx="0.0082" ixy="0.0" ixz="0.0" iyy="0.0082" iyz="0.0" izz="0.0154" />
+        </inertial>
+</link>
+<!-- Wheel Macro -->
+<xacro:macro name="wheel" params="side reflect">
+        <joint name="wheel_${side}_joint" type="continuous">
                 <parent link="base_link"/>
-                <child link="roller_link"/>
-                <origin xyz="0 -0.12 -0.04" rpy="0 0 0"/>
-        </joint>
-        <link name="roller_link">
-                <visual>
-                        <origin xyz="0 0 0" rpy="0 0 0"/>
-                        <geometry>
-                                <sphere radius="0.02"/>
-                        </geometry>
-                        <material name="black">
-                                <color rgba="0 0 0 1"/>
-                        </material>
-                </visual>
-                <collision>
-                        <origin xyz="0 0 0" rpy="0 0 0"/>
-                        <geometry>
-                                <sphere radius="0.02"/>
-                        </geometry>
-                </collision>
-                <inertial>
-                        <origin xyz="0 0 0" rpy="0 0 0"/>
-                        <mass value="0.1"/>
-                                <inertia ixx="0.0082" ixy="0.0" ixz="0.0" iyy="0.0082" iyz="0.0" izz="0.0154" />
-                </inertial>
-        </link>
-        <!-- Right wheel -->
-        <joint name="wheel_right_joint" type="continuous">
-                <parent link="base_link"/>
-                <child link="wheel_right_link"/>
-                <origin xyz="-0.11 0 -0.03" rpy="0 1.57075 0"/>
+                <child link="wheel_${side}_link"/>
+                <origin xyz="${reflect*0.11} 0 -0.03" rpy="0 1.57075 0"/>
                 <axis xyz="0 0 1"/>
         </joint>
-        <link name="wheel_right_link">
+        <link name="wheel_${side}_link">
                 <visual>
                         <origin xyz="0 0 0" rpy="0 0 0"/>
@@ -55,35 +56,9 @@
                         <origin xyz="0 0 0" rpy="0 0 0"/>
                         <mass value="0.2"/>
-                                <inertia ixx="0.0082" ixy="0.0" ixz="0.0" iyy="0.0082" iyz="0.0" izz="0.0154" />
+                        <inertia ixx="0.0082" ixy="0.0" ixz="0.0" iyy="0.0082" iyz="0.0" izz="0.0154" />
                 </inertial>
         </link>
-        <!-- Left wheel -->
-        <joint name="wheel_left_joint" type="continuous">
-                <parent link="base_link"/>
-                <child link="wheel_left_link"/>
-                <origin xyz="0.11 0 -0.03" rpy="0 1.57075 0"/>
-                <axis xyz="0 0 1"/>
-        </joint>
-        <link name="wheel_left_link">
-                <visual>
-                        <origin xyz="0 0 0" rpy="0 0 0"/>
-                        <geometry>
-                                <cylinder length="0.016" radius="0.033"/>
-                        </geometry>
-                        <material name="black">
-                                <color rgba="0 0 0 1"/>
-                        </material>
-                </visual>
-                <collision>
-                        <origin xyz="0 0 0" rpy="0 0 0"/>
-                        <geometry>
-                                <cylinder length="0.016" radius="0.033"/>
-                        </geometry>
-                </collision>
-                <inertial>
-                        <origin xyz="0 0 0" rpy="0 0 0"/>
-                        <mass value="0.2"/>
-                                <inertia ixx="0.0082" ixy="0.0" ixz="0.0" iyy="0.0082" iyz="0.0" izz="0.0154" />
-                </inertial>
-        </link>
+</xacro:macro>
+<xacro:wheel side="right" reflect="-1"/>
+<xacro:wheel side="left" reflect="1"/>
 </robot>
